File: Hardware/PROIECTUL TUL.sch (EAGLE design)
At the start: 101 parts, among them IC1 RT6160AWSC, IC2 DRV2605YZFR_DRV2605YZFR, IC3 BQ25180YBGR_BQ25180YBGR, IC4 BMA423_BMA423, J1 TC2030-IDC_TC2030-IDC, J3 503480-2400_503480-2400, J4 KH-TYPE-C-16P_KH-TYPE-C-16P, Q1 20V/4.2A/52mΩ/1.4W, Q2 SI1308EDL-T1-GE3, SW1 2025-10-22_07-23-44_LIBRARY_E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

Commit message: variantele care cred ca-s finale
Parts:
- removed SW1, SW2, SW3: 2025-10-22_07-23-44_LIBRARY_EVP-AKE31ASW_EVP-AKE31A_PAN, InkTime_v5:2025-10-22_07-23-44_LIBRARY_EVP-AKE31ASW_EVP-AKE31A_PAN
- added SW4, SW5, SW6: 2025-10-22_07-23-44_LIBRARY_EVP-AKE31A, InkTime_v5:2025-10-22_07-23-44_LIBRARY_EVP-AKE31A
- renumbered J4 to J2
Connections:
- new net N$13: J2.GND
- new net N$16: J2.DN2
- new net N$24: J2.DP2
- net DN: no longer J2.DN2
- net DP: no longer J2.DP2
- net GND: now also SW4.1, SW5.1, SW6.1; no longer J2.GND, SW1.1, SW2.1, SW3.1
- net P0.13/1.5D: now also SW4.2; no longer SW1.2
- net P0.14/1.5D: now also SW5.2; no longer SW2.2
- net P1.02/1.6C: now also SW6.2; no longer SW3.2
